File: throwing-star.sch (KiCad schematic (older format))
At the start: 6 parts, among them J1 RJ45, J2 RJ45, J3 RJ45, J4 RJ45

Commit message: update design to KiCad 5.1
Parts:
- removed J1, J2, J3, J4: RJ45, symbol RJ45
- added J1, J2, J3, J4: RJ45_Shielded, Connector_RJ:RJ45_Amphenol_RJHSE538X, symbol Connector:RJ45_Shielded
- C1, C2: footprint (none) -> Capacitor_THT:C_Disc_D5.0mm_W2.5mm_P2.50mm; symbol C -> Device:C; Description (none) -> 220pF ±10% 100V Ceramic Capacitor C0G, NP0 Radial; Manufacturer (none) -> KEMET; Part Number (none) -> C315C221K1G5TA
Connections:
- wire segments 40 -> 56
Other:
- note added: "Connectors are intended for population\nwith Amphenol RJHSE5080, but they\nmay be populated with other models\nfrom the RJHSE series. If populated\nwith a shielded model, the shields of the\nfour ports will be connected."
- note added: "J3 and J4 are guaranteed to be\nreceive-only if connected to ports\nwith Auto MDI-X disabled."
