File: throwing-star.sch (KiCad schematic (older format))
At the start: 6 parts, among them J1 RJ45_Shielded, J2 RJ45_Shielded, J3 RJ45_Shielded, J4 RJ45_Shielded

Commit message: add Throwing Star LAN Tap Pro layout
Parts:
- J1, J2, J3, J4: footprint Connector_RJ:RJ45_Amphenol_RJHSE538X -> throwing-star:RJ45_Amphenol_RJHSE538X_TSLT
Changed lines of the file:
@@
 Sheet 1 1
 Title "Throwing Star LAN Tap"
-Date "2020-07-27"
+Date "2020-07-28"
 Rev "1"
 Comp "Copyright (c) 2010-2020 Great Scott Gadgets <info@greatscottgadgets.com>"
@@
 F 0 "J1" V 4061 3230 50  0000 L CNN
 F 1 "RJ45_Shielded" V 4152 3230 50  0000 L CNN
-F 2 "Connector_RJ:RJ45_Amphenol_RJHSE538X" V 4050 2725 50  0001 C CNN
+F 2 "throwing-star:RJ45_Amphenol_RJHSE538X_TSLT" V 4050 2725 50  0001 C CNN
 F 3 "~" V 4050 2725 50  0001 C CNN
 F 4 "Amphenol" V 4050 2700 50  0001 C CNN "Manufacturer"
@@
 F 0 "J2" V 6961 3230 50  0000 L CNN
 F 1 "RJ45_Shielded" V 7052 3230 50  0000 L CNN
-F 2 "Connector_RJ:RJ45_Amphenol_RJHSE538X" V 6950 2725 50  0001 C CNN
+F 2 "throwing-star:RJ45_Amphenol_RJHSE538X_TSLT" V 6950 2725 50  0001 C CNN
 F 3 "~" V 6950 2725 50  0001 C CNN
 F 4 "Amphenol" V 6950 2700 50  0001 C CNN "Manufacturer"
@@
 F 0 "J3" V 4900 4950 50  0000 C CNN
 F 1 "RJ45_Shielded" V 4800 4950 50  0000 C CNN
-F 2 "Connector_RJ:RJ45_Amphenol_RJHSE538X" V 5250 4925 50  0001 C CNN
+F 2 "throwing-star:RJ45_Amphenol_RJHSE538X_TSLT" V 5250 4925 50  0001 C CNN
 F 3 "~" V 5250 4925 50  0001 C CNN
 F 4 "Amphenol" V 5250 4900 50  0001 C CNN "Manufacturer"
@@
 F 0 "J4" V 6100 4950 50  0000 C CNN
 F 1 "RJ45_Shielded" V 6000 4950 50  0000 C CNN
-F 2 "Connector_RJ:RJ45_Amphenol_RJHSE538X" V 6450 4925 50  0001 C CNN
+F 2 "throwing-star:RJ45_Amphenol_RJHSE538X_TSLT" V 6450 4925 50  0001 C CNN
 F 3 "~" V 6450 4925 50  0001 C CNN
 F 4 "Amphenol" V 6450 4900 50  0001 C CNN "Manufacturer"
